Commit message: fix legacy file path
Signed-off-by: wsribunm <worawissribunma@gmail.com>

File: urdf/cub1.urdf (robot description, URDF)
Before this commit: robot nvp, 1 links, 0 joints
Links:
- link cub1: geometry visual mesh filename=package://cub_description/meshes/cub_mesh.dae scale=5 5 5

File: urdf/simcub1.urdf (robot description, URDF)
Before this commit: robot nvp, 1 links, 0 joints
Links:
- removed link base_link
- added link sim; visual mesh filename=package://cub_description/meshes/cub_mesh.dae scale=5 5 5
